Commit message: Add files via upload

File: doosan-robot2/urdf/m0609_isaac_sim.urdf (robot description, URDF)
Before this commit: robot m0609, 9 links, 8 joints
Links:
- link base_link: geometry collision mesh filename=/home/rokey/cobot3_ws/isaacpjt/M0609/doosan-robot2/urdf/mes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 scale=0.001 0.001 0.001; visual mesh filename=/home/rokey/cobot3_ws/isaacpjt/M0609/doosan-robot2/urdf/mes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 scale=0.001 0.001 0.001
- link link_1: geometry collision mesh filename=/home/rokey/cobot3_ws/isaacpjt/M0609/doosan-robot2/urdf/mes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 scale=0.001 0.001 0.001; visual mesh filename=/home/rokey/cobot3_ws/isaacpjt/M0609/doosan-robot2/urdf/mes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 scale=0.001 0.001 0.001
- link link_2: geometry collision mesh filename=/home/rokey/cobot3_ws/isaacpjt/M0609/doosan-robot2/urdf/mes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 scale=0.001 0.001 0.001; collision mesh filename=/home/rokey/cobot3_ws/isaacpjt/M0609/doosan-robot2/urdf/mes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 scale=0.001 0.001 0.001
- link link_3: geometry collision mesh filename=/home/rokey/cobot3_ws/isaacpjt/M0609/doosan-robot2/urdf/mes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 scale=0.001 0.001 0.001; visual mesh filename=/home/rokey/cobot3_ws/isaacpjt/M0609/doosan-robot2/urdf/mes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 scale=0.001 0.001 0.001
- link link_4: geometry collision mesh filename=/home/rokey/cobot3_ws/isaacpjt/M0609/doosan-robot2/urdf/mes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 scale=0.001 0.001 0.001; collision mesh filename=/home/rokey/cobot3_ws/isaacpjt/M0609/doosan-robot2/urdf/mes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 scale=0.001 0.001 0.001
- link link_5: geometry collision mesh filename=/home/rokey/cobot3_ws/isaacpjt/M0609/doosan-robot2/urdf/mes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 scale=0.001 0.001 0.001; visual mesh filename=/home/rokey/cobot3_ws/isaacpjt/M0609/doosan-robot2/urdf/mes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 scale=0.001 0.001 0.001
- link link_6: geometry collision mesh filename=/home/rokey/cobot3_ws/isaacpjt/M0609/doosan-robot2/urdf/mes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 scale=0.001 0.001 0.001; visual mesh filename=/home/rokey/cobot3_ws/isaacpjt/M0609/doosan-robot2/urdf/mes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 scale=0.001 0.001 0.001
